Commit message: update

File: examples/arx_ros2/urdf/X7S_arm_only.urdf (robot description, URDF)
Before this commit: robot X7S, 23 links, 22 joints
Joints:
- joint joint15: limit lower=-10 upper=10 effort=100 velocity=1000 -> lower=-0.1 upper=0.3 effort=100 velocity=1000
- joint joint6: limit lower=-10 upper=10 effort=100 velocity=1000 -> lower=-0.3 upper=0.1 effort=100 velocity=1000
